File: Battery_Indicator.sch (EAGLE design)
At the start: 33 parts, among them IC1 MEGA8-AI, IC2 7805DT, Q1 IRF3704S, Q2 IRF3704S

Commit message: Update EAGLE project files
Parts:
- added GND, MISO, SCK: (no value), wirepad:SMD2
- C3: device rcl:CPOL-EUE2-4 -> rcl:CPOL-EUSMCD
- IC1: value MEGA8-AI -> ATMEGA8
- LED1: value RED 1st -> (none); device led:LED3MM -> wirepad:SMD2
- LED2: value GREEN 2nd -> (none); device led:LED3MM -> wirepad:SMD2
- LED3: value GREEN 3rd -> (none); device led:LED3MM -> wirepad:SMD2
- LED4: value GREEN 4th -> (none); device led:LED3MM -> wirepad:SMD2
- LED5: value GREEN 5th -> (none); device led:LED3MM -> wirepad:SMD2
- renumbered COPTER_VCC_1 to COPTER_VCC, COPTER_VCC_2 to COPTER_GND, USART_RX to RX, USART_TX to TX
Connections:
- new net N$25: IC1.PB4(MISO), MISO.P
- new net N$26: IC1.PB5(SCK), SCK.P
- net GND: now also GND.P; no longer LED1.C, LED2.C, LED3.C, LED4.C, LED5.C
- net N$10: now also LED4.P; no longer LED4.A
- net N$11: now also LED5.P; no longer LED5.A
- net N$7: now also LED1.P; no longer LED1.A
- net N$8: now also LED2.P; no longer LED2.A
- net N$9: now also LED3.P; no longer LED3.A
